Commit message: feat: True 4WIS/4WID swerve controller, asymmetric slope leveling, look-ahead terrain perception, and test suite

File: src/rover_description/urdf/rover.urdf (robot description, URDF)
Before this commit: robot hex_tele_rover, 106 links, 105 joints
Joints:
- joint legBL_steer_joint: limit lower=-0.65 upper=0.65 effort=50.0 velocity=3.0 -> lower=-3.14159 upper=3.14159 effort=50.0 velocity=3.0
- joint legBR_steer_joint: limit lower=-0.65 upper=0.65 effort=50.0 velocity=3.0 -> lower=-3.14159 upper=3.14159 effort=50.0 velocity=3.0
- joint legFL_steer_joint: limit lower=-0.65 upper=0.65 effort=50.0 velocity=3.0 -> lower=-3.14159 upper=3.14159 effort=50.0 velocity=3.0
- joint legFR_steer_joint: limit lower=-0.65 upper=0.65 effort=50.0 velocity=3.0 -> lower=-3.14159 upper=3.14159 effort=50.0 velocity=3.0
